File: hw/KEY_ARRAY.kicad_sch (KiCad schematic)
At the start: 64 parts, among them U5 74HC595

Commit message: Schematic updated.
Connections:
- net GP5 renamed C5
Changed lines of the file:
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@@
   (junction (at 50.8 21.59) (diameter 0) (color 0 0 0 0)
   )
+  (junction (at 167.64 85.09) (diameter 0) (color 0 0 0 0)
+  )
   (junction (at 76.2 57.15) (diameter 0) (color 0 0 0 0)
   )
@@
   )
   (junction (at 167.64 43.18) (diameter 0) (color 0 0 0 0)
+  )
+  (junction (at 20.32 71.12) (diameter 0) (color 0 0 0 0)
+  )
+  (junction (at 20.32 85.09) (diameter 0) (color 0 0 0 0)
   )
   (junction (at 81.28 21.59) (diameter 0) (color 0 0 0 0)
@@
     (stroke (width 0) (type default))
   )
-  (wire (pts (xy 167.64 57.15) (xy 167.64 90.17))
+  (wire (pts (xy 167.64 57.15) (xy 167.64 85.09))
     (stroke (width 0) (type default))
   )
@@
     (stroke (width 0) (type default))
   )
+  (wire (pts (xy 17.78 85.09) (xy 20.32 85.09))
+    (stroke (width 0) (type default))
+  )
   (wire (pts (xy 106.68 29.21) (xy 106.68 43.18))
     (stroke (width 0) (type default))
@@
     (stroke (width 0) (type default))
   )
+  (wire (pts (xy 167.64 85.09) (xy 170.18 85.09))
+    (stroke (width 0) (type default))
+  )
   (wire (pts (xy 50.8 63.5) (xy 50.8 71.12))
     (stroke (width 0) (type default))
@@
     (stroke (width 0) (type default))
   )
+  (wire (pts (xy 17.78 71.12) (xy 20.32 71.12))
+    (stroke (width 0) (type default))
+  )
   (wire (pts (xy 81.28 43.18) (xy 81.28 35.56))
     (stroke (width 0) (type default))
@@
   )
   (wire (pts (xy 193.04 116.84) (xy 196.85 116.84))
+    (stroke (width 0) (type default))
+  )
+  (wire (pts (xy 167.64 85.09) (xy 167.64 90.17))
     (stroke (width 0) (type default))
   )
@@
     )
   )
+  (global_label "C5" (shape input) (at 170.18 85.09 0) (fields_autoplaced)
+    (effects (font (size 1.27 1.27)) (justify left))
+    (property "Intersheetrefs" "${INTERSHEET_REFS}" (at 175.6447 85.09 0)
+      (effects (font (size 1.27 1.27)) (justify left) hide)
+    )
+  )
+  (global_label "R5" (shape input) (at 17.78 85.09 180) (fields_autoplaced)
+    (effects (font (size 1.27 1.27)) (justify right))
+    (property "Intersheetrefs" "${INTERSHEET_REFS}" (at 12.3153 85.09 0)
+      (effects (font (size 1.27 1.27)) (justify right) hide)
+    )
+  )
   (global_label "GP1" (shape input) (at 193.04 99.06 180) (fields_autoplaced)
     (effects (font (size 1.27 1.27)) (justify right))
@@
       (effects (font (size 1.27 1.27)) (justify right) hide)
     )
+  )
+  (global_label "R4" (shape input) (at 17.78 71.12 180) (fields_autoplaced)
+    (effects (font (size 1.27 1.27)) (justify right))
+    (property "Intersheetrefs" "${INTERSHEET_REFS}" (at 12.3153 71.12 0)
+      (effects (font (size 1.27 1.27)) (justify right) hide)
+    )
