File: hw/RP2040_KBD.kicad_pcb (KiCad board)
At the start: 2 copper layers, 106.5 x 125.4 mm, 124 parts, among them J1 BAT_9V, J2 SWD, J3 USB_C_Receptacle_USB2.0, J4 TFT_LCD, Q1 2N7002, SW1 SW_Push, U1 AMS1117-5.0, U2 XC6220B331MR, U3 W25Q128JVSS, U4 RP2040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

Commit message: Schematic updated.
Parts:
- removed C21, C22: 100nF, Capacitor_SMD:C_0603_1608Metric
- removed R30, R31: 10k, Resistor_SMD:R_0603_1608Metric
- removed R32, R33: 100k, Resistor_SMD:R_0603_1608Metric
- added D29: 1N4148WS, Diode_SMD:D_SOD-323, F.Cu at (122.6, 49.3)
- added D30: 1N4148WS, Diode_SMD:D_SOD-323, F.Cu at (141.6, 49.3)
Connections:
- net GP5 renamed C5
- SW24 pad 1: Net-(R30-Pad2) -> GP3
- SW24 pad 2: +3V3 -> Net-(D29-A)
- SW25 pad 1: Net-(R31-Pad2) -> GP4
- SW25 pad 2: +3V3 -> Net-(D30-A)
Routing:
- net GP4: track 219.3 -> 339.3 mm, vias 2 -> 3
- net GP3: track 215.6 -> 327.2 mm, vias 2 -> 3
- net GP13: track 47.5 -> 0.00 mm, vias 2 -> 0
- net C5: track 160.1 -> 190.1 mm, vias 2 -> 4
- net Net-(D29-A): track 0.00 -> 27.6 mm
- net Net-(D30-A): track 0.00 -> 27.6 mm
- net Net-(R31-Pad2): track 26.5 -> 0.00 mm
- net Net-(R30-Pad2): track 26.4 -> 0.00 mm
- net +3V3: track 385.5 -> 366.0 mm, vias 18 -> 17
- net GND: track 367.2 -> 353.6 mm, vias 369 -> 384
- net GP22: track 3.00 -> 0.00 mm
- net SWD_3V3: track 27.1 -> 25.6 mm, vias 0 -> 2
- net GP2: track 260.7 -> 259.7 mm, vias 3 -> 4
- net BAT_5V: track 31.6 -> 30.8 mm
